File: PCB/pcb project.brd (EAGLE design)
At the start: 56.2 x 60.1 mm, 9 parts

Commit message: Finalized PCB design + wind tunnel analysis, MCU code still a mess
Parts:
- removed D1, D4: (no value), adafruit:SOD-323F
- removed R1: 1k, adafruit:R0603
- removed R2, R4: 2k, adafruit:R0603
- moved SD_CARD 1.27 mm to (21.6, 45.7), flipped to the bottom
Connections:
- removed net 3V: MS1.2, R1.2
- removed net N$2: D1.C, DLLR-L10G-E1BD-C-NAV8_BOT.3, MS1.19, R2.1
- removed net SCL: DLLR-L10G-E1BD-C-NAV8_BOT.4, DLLR-L10G-E1BD-C-NAV8_TOP.4, MS1.18, R1.1
- removed net SDA: D1.A, D4.A, MS1.17, R2.2, R4.2
- removed net TOP_DIS: D4.C, DLLR-L10G-E1BD-C-NAV8_TOP.3, MS1.20, R4.1
- new net SENSORSELECT1: DLLR-L10G-E1BD-C-NAV8_TOP.8, MS1.23
- new net SENSORSELECT2: DLLR-L10G-E1BD-C-NAV8_BOT.8, MS1.24
- net MISO: now also DLLR-L10G-E1BD-C-NAV8_BOT.6, DLLR-L10G-E1BD-C-NAV8_TOP.6
- net MOSI: now also DLLR-L10G-E1BD-C-NAV8_BOT.3, DLLR-L10G-E1BD-C-NAV8_TOP.3
- net SCK: now also DLLR-L10G-E1BD-C-NAV8_BOT.4, DLLR-L10G-E1BD-C-NAV8_TOP.4
- net VCC: now also MS1.2
Routing:
- net VCC: track 50.9 -> 0.00 mm
- net N$2: track 45.0 -> 0.00 mm, vias 1 -> 0
- net SCL: track 44.3 -> 0.00 mm
- net 3V: track 39.0 -> 0.00 mm
- net TOP_DIS: track 31.7 -> 0.00 mm, vias 2 -> 0
- net MISO: track 45.7 -> 74.6 mm, vias 1 -> 0
- net SDA: track 24.3 -> 0.00 mm
- net SENSORSELECT1: track 0.00 -> 23.8 mm
- net SENSORSELECT2: track 0.00 -> 19.0 mm
- net SCK: track 49.5 -> 58.5 mm, vias 1 -> 0
- net MOSI: track 62.1 -> 56.0 mm, vias 1 -> 2
- net GND: track 4.22 -> 1.29 mm, vias 2 -> 1
- added copper zone on layer 16, net VCC
Other:
- outline, holes or cut-outs redrawn
