File: PCB/pcb project.sch (EAGLE design)
At the start: 9 parts

Commit message: Finalized PCB design + wind tunnel analysis, MCU code still a mess
Parts:
- removed D1, D4: (no value), adafruit:DIODESOD-323F
- removed R1: 1k, adafruit:R-US_R0603
- removed R2, R4: 2k, adafruit:R-US_R0603
Connections:
- removed net 3V: MS1.3V, R1.2
- removed net N$2: D1.C, DLLR-L10G-E1BD-C-NAV8_BOT.SDA/MOSI, MS1.GPIO5, R2.1
- removed net SCL: DLLR-L10G-E1BD-C-NAV8_BOT.SCL/SCLK, DLLR-L10G-E1BD-C-NAV8_TOP.SCL/SCLK, MS1.GPIOSCL, R1.1
- removed net SDA: D1.A, D4.A, MS1.GPIOSDA, R2.2, R4.2
- removed net TOP_DIS: D4.C, DLLR-L10G-E1BD-C-NAV8_TOP.SDA/MOSI, MS1.GPIO6, R4.1
- new net SENSORSELECT1: DLLR-L10G-E1BD-C-NAV8_TOP./SS, MS1.GPIO11
- new net SENSORSELECT2: DLLR-L10G-E1BD-C-NAV8_BOT./SS, MS1.GPIO12
- net MISO: now also DLLR-L10G-E1BD-C-NAV8_BOT.MISO, DLLR-L10G-E1BD-C-NAV8_TOP.MISO
- net MOSI: now also DLLR-L10G-E1BD-C-NAV8_BOT.SDA/MOSI, DLLR-L10G-E1BD-C-NAV8_TOP.SDA/MOSI
- net SCK: now also DLLR-L10G-E1BD-C-NAV8_BOT.SCL/SCLK, DLLR-L10G-E1BD-C-NAV8_TOP.SCL/SCLK
- net VCC: now also MS1.3V
Other:
- note added: "Busby & Diamond"
- note added: "June 29, 2020"
- note added: "REV 1.0"
- note removed: "January 8, 2020"
